Commit message: fixed some naming

File: franka_description/robots/drill_old.xacro (robot description, xacro)
@@ -1,17 +1,17 @@
 <?xml version="1.0" encoding="utf-8"?>
-<robot xmlns:xacro="http://www.ros.org/wiki/xacro" name="driller_new">
+<robot xmlns:xacro="http://www.ros.org/wiki/xacro" name="drill_old">
   <!-- safety_distance: Minimum safety distance in [m] by which the collision volumes are expanded and which is enforced during robot motions -->
-  <xacro:macro name="driller_new" params="connected_to:='' ns:='' rpy:='0 0 0' xyz:='0 0 0' safety_distance:=0">
+  <xacro:macro name="drill_old" params="connected_to:='' ns:='' rpy:='0 0 0' xyz:='0 0 0' safety_distance:=0">
     <xacro:unless value="${connected_to == ''}">
-      <joint name="${ns}_driller_new_joint" type="fixed">
+      <joint name="${ns}_drill_old_joint" type="fixed">
         <parent link="${connected_to}"/>
-        <child link="${ns}_driller_new"/>
+        <child link="${ns}_drill_old"/>
         <origin xyz="${xyz}" rpy="${rpy}"/>
       </joint>
     </xacro:unless>
-    <link name="${ns}_driller_new">
+    <link name="${ns}_drill_old">
       <visual>
         <geometry>
-          <mesh filename="package://franka_description/meshes/visual/driller_new_m.stl"/>
+          <mesh filename="package://franka_description/meshes/visual/drill_old.stl"/>
         </geometry>
       </visual>

File: franka_description/robots/panda_arm_drill_old.urdf.xacro (robot description, xacro)
@@ -3,6 +3,6 @@
 <link name="world" />
   <xacro:include filename="$(find franka_description)/robots/panda_arm.xacro"/>
-  <xacro:include filename="$(find franka_description)/robots/driller_new.xacro"/>
+  <xacro:include filename="$(find franka_description)/robots/drill_old.xacro"/>
 <xacro:panda_arm safety_distance="0.03" connected_to="world"/>
-<xacro:driller_new ns="panda" rpy="0 0 0.785398" connected_to="panda_link8" safety_distance="0.03"/>
+<xacro:drill_old ns="panda" rpy="0 0 0.785398" connected_to="panda_link8" safety_distance="0.03"/>
 </robot>

Commit message: added self collision avoidance

File: franka_description/robots/drill_old.xacro (robot description, xacro)
@@ -18,6 +18,8 @@
       <collision>
         <origin rpy="0 0 0" xyz="0 -0.051 0.0425"/>
+<!--         <origin rpy="0 0 0" xyz="0 0.3 0.0425"/> -->
         <geometry>
             <box size="0.082 0.25 0.09"/>
+<!--             <box size="0.082 0.6 0.09"/> -->
         </geometry>
     </collision>
